Commit message: change joint name

File: urdf/allegro_hand_description_right.urdf.xacro (robot description, xacro)
@@ -101,5 +101,5 @@
     	</collision>
 	</link>
-	<joint name="THJ0" type="revolute">
+	<joint name="THJ_0" type="revolute">
     	<axis xyz="-1 0 0"/>
     	<limit effort="0" velocity="0" lower="${limit_0_t_low-joint_safety_margin}" upper="${limit_0_t_up-joint_safety_margin}" />
@@ -125,5 +125,5 @@
 		</collision>
 	</link>
-  	<joint name="THJ1" type="revolute">
+  	<joint name="THJ_1" type="revolute">
     	<axis xyz="0 0 1"/>
      	<limit effort="0" velocity="0" lower="${limit_1_t_low+joint_safety_margin}" upper="${limit_1_t_up-joint_safety_margin}" />
@@ -151,5 +151,5 @@
 		</collision>
 	</link>
-  <joint name="THJ2" type="revolute">
+  <joint name="THJ_2" type="revolute">
 		<axis xyz="0 1 0"/>
 		<limit effort="0" velocity="0" lower="${limit_2_t_low+joint_safety_margin}" upper="${limit_2_t_up-joint_safety_margin}" />
@@ -174,5 +174,5 @@
     	</collision>
 	</link>
-	<joint name="THJ3" type="revolute">
+	<joint name="THJ_3" type="revolute">
     	<axis xyz="0 1 0"/>
      	<limit effort="0" velocity="0" lower="${limit_3_t_low+joint_safety_margin}" upper="${limit_3_t_up-joint_safety_margin}" />
