Commit message: euslisp FJT failed if velocity is set to 0 (don't know real value, set it to 1)

File: urdf/allegro_hand_description_left.urdf (robot description, URDF)
Before this commit: robot allegro_hand_left, 21 links, 20 joints
Joints:
- joint joint_0.0: limit lower=-0.47 upper=0.47 effort=0 velocity=0 -> lower=-0.47 upper=0.47 effort=0 velocity=1
- joint joint_1.0: limit lower=-0.196 upper=1.61 effort=0 velocity=0 -> lower=-0.196 upper=1.61 effort=0 velocity=1
- joint joint_10.0: limit lower=-0.174 upper=1.709 effort=0 velocity=0 -> lower=-0.174 upper=1.709 effort=0 velocity=1
- joint joint_11.0: limit lower=-0.227 upper=1.618 effort=0 velocity=0 -> lower=-0.227 upper=1.618 effort=0 velocity=1
- joint joint_12.0: limit lower=0.263 upper=1.396 effort=0 velocity=0 -> lower=0.263 upper=1.396 effort=0 velocity=1
- joint joint_13.0: limit lower=-0.105 upper=1.163 effort=0 velocity=0 -> lower=-0.105 upper=1.163 effort=0 velocity=1
- joint joint_14.0: limit lower=-0.189 upper=1.644 effort=0 velocity=0 -> lower=-0.189 upper=1.644 effort=0 velocity=1
- joint joint_15.0: limit lower=-0.162 upper=1.719 effort=0 velocity=0 -> lower=-0.162 upper=1.719 effort=0 velocity=1
- joint joint_2.0: limit lower=-0.174 upper=1.709 effort=0 velocity=0 -> lower=-0.174 upper=1.709 effort=0 velocity=1
- joint joint_3.0: limit lower=-0.227 upper=1.618 effort=0 velocity=0 -> lower=-0.227 upper=1.618 effort=0 velocity=1
- joint joint_4.0: limit lower=-0.47 upper=0.47 effort=0 velocity=0 -> lower=-0.47 upper=0.47 effort=0 velocity=1
- joint joint_5.0: limit lower=-0.196 upper=1.61 effort=0 velocity=0 -> lower=-0.196 upper=1.61 effort=0 velocity=1
- joint joint_6.0: limit lower=-0.174 upper=1.709 effort=0 velocity=0 -> lower=-0.174 upper=1.709 effort=0 velocity=1
- joint joint_7.0: limit lower=-0.227 upper=1.618 effort=0 velocity=0 -> lower=-0.227 upper=1.618 effort=0 velocity=1
- joint joint_8.0: limit lower=-0.47 upper=0.47 effort=0 velocity=0 -> lower=-0.47 upper=0.47 effort=0 velocity=1
- joint joint_9.0: limit lower=-0.196 upper=1.61 effort=0 velocity=0 -> lower=-0.196 upper=1.61 effort=0 velocity=1

File: urdf/allegro_hand_description_left.urdf.xacro (robot description, xacro)
@@ -154,5 +154,5 @@
 	<joint name="joint_${finger_num*4+0}" type="revolute">
     	<axis xyz="+1 0 0"/>
-    	<limit effort="0" velocity="0" lower="${limit_0_t_low-joint_safety_margin}" upper="${limit_0_t_up-joint_safety_margin}" />
+    	<limit effort="0" velocity="1" lower="${limit_0_t_low-joint_safety_margin}" upper="${limit_0_t_up-joint_safety_margin}" />
     	<parent link="base_link"/>
     	<child link="link_${finger_num*4+0}"/>
@@ -178,5 +178,5 @@
   	<joint name="joint_${finger_num*4+1}" type="revolute">
     	<axis xyz="0 0 -1"/>
-     	<limit effort="0" velocity="0" lower="${limit_1_t_low+joint_safety_margin}" upper="${limit_1_t_up-joint_safety_margin}" />
+     	<limit effort="0" velocity="1" lower="${limit_1_t_low+joint_safety_margin}" upper="${limit_1_t_up-joint_safety_margin}" />
     	<parent link="link_${finger_num*4+0}"/>
     	<child link="link_${finger_num*4+1}"/>
@@ -204,5 +204,5 @@
   <joint name="joint_${finger_num*4+2}" type="revolute">
 		<axis xyz="0 1 0"/>
-		<limit effort="0" velocity="0" lower="${limit_2_t_low+joint_safety_margin}" upper="${limit_2_t_up-joint_safety_margin}" />
+		<limit effort="0" velocity="1" lower="${limit_2_t_low+joint_safety_margin}" upper="${limit_2_t_up-joint_safety_margin}" />
 		<parent link="link_${finger_num*4+1}"/>
 		<child link="link_${finger_num*4+2}"/>
@@ -227,5 +227,5 @@
 	<joint name="joint_${finger_num*4+3}" type="revolute">
     	<axis xyz="0 1 0"/>
-     	<limit effort="0" velocity="0" lower="${limit_3_t_low+joint_safety_margin}" upper="${limit_3_t_up-joint_safety_margin}" />
+     	<limit effort="0" velocity="1" lower="${limit_3_t_low+joint_safety_margin}" upper="${limit_3_t_up-joint_safety_margin}" />
     	<parent link="link_${finger_num*4+2}"/>
     	<child link="link_${finger_num*4+3}"/>
@@ -275,5 +275,5 @@
   	<joint name="joint_${finger_num*4+0}" type="revolute">
     	<axis xyz="0 0 1"/>
-    	<limit effort="0" velocity="0" lower="${limit_0_low+joint_safety_margin}" upper="${limit_0_up-joint_safety_margin}" />
+    	<limit effort="0" velocity="1" lower="${limit_0_low+joint_safety_margin}" upper="${limit_0_up-joint_safety_margin}" />
     	<parent link="base_link"/>
     	<child link="link_${finger_num*4+0}"/>
@@ -296,5 +296,5 @@
   	</link>
   	<joint name="joint_${finger_num*4+1}" type="revolute">
-  		<limit effort="0" velocity="0" lower="${limit_1_low+joint_safety_margin}" upper="${limit_1_up-joint_safety_margin}" />
+  		<limit effort="0" velocity="1" lower="${limit_1_low+joint_safety_margin}" upper="${limit_1_up-joint_safety_margin}" />
     	<axis xyz="0 1 0"/>
     	<parent link="link_${finger_num*4+0}"/>
@@ -319,5 +319,5 @@
   	<joint name="joint_${finger_num*4+2}" type="revolute">
     	<axis xyz="0 1 0"/>
-    	<limit effort="0" velocity="0" lower="${limit_2_low+joint_safety_margin}" upper="${limit_2_up-joint_safety_margin}" />
+    	<limit effort="0" velocity="1" lower="${limit_2_low+joint_safety_margin}" upper="${limit_2_up-joint_safety_margin}" />
     	<parent link="link_${finger_num*4+1}"/>
     	<child link="link_${finger_num*4+2}"/>
@@ -341,5 +341,5 @@
   	<joint name="joint_${finger_num*4+3}" type="revolute">
     	<axis xyz="0 1 0"/>
-    	<limit effort="0" velocity="0" lower="${limit_3_low+joint_safety_margin}" upper="${limit_3_up-joint_safety_margin}" />
+    	<limit effort="0" velocity="1" lower="${limit_3_low+joint_safety_margin}" upper="${limit_3_up-joint_safety_margin}" />
     	<parent link="link_${finger_num*4+2}"/>
     	<child link="link_${finger_num*4+3}"/>

File: urdf/allegro_hand_description_right.urdf (robot description, URDF)
Before this commit: robot allegro_hand_right, 21 links, 20 joints
Joints:
- joint joint_0.0: limit lower=-0.47 upper=0.47 effort=0 velocity=0 -> lower=-0.47 upper=0.47 effort=0 velocity=1
- joint joint_1.0: limit lower=-0.196 upper=1.61 effort=0 velocity=0 -> lower=-0.196 upper=1.61 effort=0 velocity=1
- joint joint_10.0: limit lower=-0.174 upper=1.709 effort=0 velocity=0 -> lower=-0.174 upper=1.709 effort=0 velocity=1
- joint joint_11.0: limit lower=-0.227 upper=1.618 effort=0 velocity=0 -> lower=-0.227 upper=1.618 effort=0 velocity=1
- joint joint_12.0: limit lower=0.263 upper=1.396 effort=0 velocity=0 -> lower=0.263 upper=1.396 effort=0 velocity=1
- joint joint_13.0: limit lower=-0.105 upper=1.163 effort=0 velocity=0 -> lower=-0.105 upper=1.163 effort=0 velocity=1
- joint joint_14.0: limit lower=-0.189 upper=1.644 effort=0 velocity=0 -> lower=-0.189 upper=1.644 effort=0 velocity=1
- joint joint_15.0: limit lower=-0.162 upper=1.719 effort=0 velocity=0 -> lower=-0.162 upper=1.719 effort=0 velocity=1
- joint joint_2.0: limit lower=-0.174 upper=1.709 effort=0 velocity=0 -> lower=-0.174 upper=1.709 effort=0 velocity=1
- joint joint_3.0: limit lower=-0.227 upper=1.618 effort=0 velocity=0 -> lower=-0.227 upper=1.618 effort=0 velocity=1
- joint joint_4.0: limit lower=-0.47 upper=0.47 effort=0 velocity=0 -> lower=-0.47 upper=0.47 effort=0 velocity=1
- joint joint_5.0: limit lower=-0.196 upper=1.61 effort=0 velocity=0 -> lower=-0.196 upper=1.61 effort=0 velocity=1
- joint joint_6.0: limit lower=-0.174 upper=1.709 effort=0 velocity=0 -> lower=-0.174 upper=1.709 effort=0 velocity=1
- joint joint_7.0: limit lower=-0.227 upper=1.618 effort=0 velocity=0 -> lower=-0.227 upper=1.618 effort=0 velocity=1
- joint joint_8.0: limit lower=-0.47 upper=0.47 effort=0 velocity=0 -> lower=-0.47 upper=0.47 effort=0 velocity=1
- joint joint_9.0: limit lower=-0.196 upper=1.61 effort=0 velocity=0 -> lower=-0.196 upper=1.61 effort=0 velocity=1

File: urdf/allegro_hand_description_right.urdf.xacro (robot description, xacro)
@@ -103,5 +103,5 @@
 	<joint name="THJ_0" type="revolute">
     	<axis xyz="-1 0 0"/>
-    	<limit effort="0" velocity="0" lower="${limit_0_t_low-joint_safety_margin}" upper="${limit_0_t_up-joint_safety_margin}" />
+    	<limit effort="0" velocity="1" lower="${limit_0_t_low-joint_safety_margin}" upper="${limit_0_t_up-joint_safety_margin}" />
     	<parent link="base_link"/>
     	<child link="thu_link_0"/>
@@ -127,5 +127,5 @@
   	<joint name="THJ_1" type="revolute">
     	<axis xyz="0 0 1"/>
-     	<limit effort="0" velocity="0" lower="${limit_1_t_low+joint_safety_margin}" upper="${limit_1_t_up-joint_safety_margin}" />
+     	<limit effort="0" velocity="1" lower="${limit_1_t_low+joint_safety_margin}" upper="${limit_1_t_up-joint_safety_margin}" />
     	<parent link="thu_link_0"/>
     	<child link="thu_link_1"/>
@@ -153,5 +153,5 @@
   <joint name="THJ_2" type="revolute">
 		<axis xyz="0 1 0"/>
-		<limit effort="0" velocity="0" lower="${limit_2_t_low+joint_safety_margin}" upper="${limit_2_t_up-joint_safety_margin}" />
+		<limit effort="0" velocity="1" lower="${limit_2_t_low+joint_safety_margin}" upper="${limit_2_t_up-joint_safety_margin}" />
 		<parent link="thu_link_1"/>
 		<child link="thu_link_2"/>
@@ -176,5 +176,5 @@
 	<joint name="THJ_3" type="revolute">
     	<axis xyz="0 1 0"/>
-     	<limit effort="0" velocity="0" lower="${limit_3_t_low+joint_safety_margin}" upper="${limit_3_t_up-joint_safety_margin}" />
+     	<limit effort="0" velocity="1" lower="${limit_3_t_low+joint_safety_margin}" upper="${limit_3_t_up-joint_safety_margin}" />
     	<parent link="thu_link_2"/>
     	<child link="thu_link_3"/>
@@ -224,5 +224,5 @@
   	<joint name="${j_prefix}_0" type="revolute">
     	<axis xyz="0 0 1"/>
-    	<limit effort="0" velocity="0" lower="${limit_0_low+joint_safety_margin}" upper="${limit_0_up-joint_safety_margin}" />
+    	<limit effort="0" velocity="1" lower="${limit_0_low+joint_safety_margin}" upper="${limit_0_up-joint_safety_margin}" />
     	<parent link="base_link"/>
     	<child link="${l_prefix}_0"/>
@@ -245,5 +245,5 @@
   	</link>
   	<joint name="${j_prefix}_1" type="revolute">
-  		<limit effort="0" velocity="0" lower="${limit_1_low+joint_safety_margin}" upper="${limit_1_up-joint_safety_margin}" />
+  		<limit effort="0" velocity="1" lower="${limit_1_low+joint_safety_margin}" upper="${limit_1_up-joint_safety_margin}" />
     	<axis xyz="0 1 0"/>
     	<parent link="${l_prefix}_0"/>
@@ -268,5 +268,5 @@
   	<joint name="${j_prefix}_2" type="revolute">
     	<axis xyz="0 1 0"/>
-    	<limit effort="0" velocity="0" lower="${limit_2_low+joint_safety_margin}" upper="${limit_2_up-joint_safety_margin}" />
+    	<limit effort="0" velocity="1" lower="${limit_2_low+joint_safety_margin}" upper="${limit_2_up-joint_safety_margin}" />
     	<parent link="${l_prefix}_1"/>
     	<child link="${l_prefix}_2"/>
@@ -290,5 +290,5 @@
   	<joint name="${j_prefix}_3" type="revolute">
     	<axis xyz="0 1 0"/>
-    	<limit effort="0" velocity="0" lower="${limit_3_low+joint_safety_margin}" upper="${limit_3_up-joint_safety_margin}" />
+    	<limit effort="0" velocity="1" lower="${limit_3_low+joint_safety_margin}" upper="${limit_3_up-joint_safety_margin}" />
     	<parent link="${l_prefix}_2"/>
     	<child link="${l_prefix}_3"/>
